File: Singe_transistor_AMP/Singe_transistor_AMP.sch (KiCad schematic (older format))
At the start: 11 parts, among them J1 Conn_01x03, J2 Conn_01x02, Q1 NPN

Commit message: Pie Single_transistor_AMP pievienotas komponensu datulapas un NET fails
Parts:
- C1, C3: value 40uF -> 10uF
- C2: value 40uF -> 470uF
Other:
- moved on the sheet: C3, J2
Changed lines of the file:
@@
 EESchema Schematic File Version 4
+LIBS:Singe_transistor_AMP-cache
 EELAYER 30 0
 EELAYER END
@@
 P 4550 3600
 F 0 "C1" V 4779 3600 50  0000 C CNN
-F 1 "40uF" V 4688 3600 50  0000 C CNN
+F 1 "10uF" V 4688 3600 50  0000 C CNN
 F 2 "Capacitor_THT:CP_Radial_D6.3mm_P2.50mm" H 4550 3600 50  0001 C CNN
-F 3 "~" H 4550 3600 50  0001 C CNN
+F 3 "http://www.farnell.com/datasheets/1700589.pdf" H 4550 3600 50  0001 C CNN
 	1    4550 3600
 	0    -1   -1   0
@@
 	4150 3600 4450 3600
 Wire Wire Line
-	6000 3500 5900 3500
+	5650 3450 5550 3450
 $Comp
 L Device:C_Small C3
 U 1 1 5DC28E4B
-P 5650 3400
-F 0 "C3" V 5879 3400 50  0000 C CNN
-F 1 "40uF" V 5788 3400 50  0000 C CNN
-F 2 "Capacitor_THT:CP_Radial_D6.3mm_P2.50mm" H 5650 3400 50  0001 C CNN
-F 3 "~" H 5650 3400 50  0001 C CNN
-	1    5650 3400
+P 5400 3350
+F 0 "C3" V 5629 3350 50  0000 C CNN
+F 1 "10uF" V 5538 3350 50  0000 C CNN
+F 2 "Capacitor_THT:CP_Radial_D6.3mm_P2.50mm" H 5400 3350 50  0001 C CNN
+F 3 "http://www.farnell.com/datasheets/1700589.pdf" H 5400 3350 50  0001 C CNN
+	1    5400 3350
 	0    -1   -1   0
 $EndComp
@@
 F 1 "NPN" H 5141 3555 50  0000 L CNN
 F 2 "Package_TO_SOT_THT:TO-92" H 5150 3700 50  0001 C CNN
-F 3 "~" H 4950 3600 50  0001 C CNN
+F 3 "https://www.sparkfun.com/datasheets/Components/BC546.pdf" H 4950 3600 50  0001 C CNN
 	1    4950 3600
 	1    0    0    -1
@@
 F 1 "39k" H 4809 3305 50  0000 L CNN
 F 2 "Resistor_THT:R_Axial_DIN0207_L6.3mm_D2.5mm_P5.08mm_Vertical" H 4750 3350 50  0001 C CNN
-F 3 "~" H 4750 3350 50  0001 C CNN
+F 3 "http://www.farnell.com/datasheets/2049325.pdf" H 4750 3350 50  0001 C CNN
 	1    4750 3350
 	1    0    0    -1
@@
 F 1 "10k" H 4809 3805 50  0000 L CNN
 F 2 "Resistor_THT:R_Axial_DIN0207_L6.3mm_D2.5mm_P5.08mm_Vertical" H 4750 3850 50  0001 C CNN
-F 3 "~" H 4750 3850 50  0001 C CNN
+F 3 "http://www.farnell.com/datasheets/2049325.pdf" H 4750 3850 50  0001 C CNN
 	1    4750 3850
 	1    0    0    -1
@@
 F 1 "560" H 5150 4100 50  0000 L CNN
 F 2 "Resistor_THT:R_Axial_DIN0207_L6.3mm_D2.5mm_P5.08mm_Vertical" H 5050 4050 50  0001 C CNN
-F 3 "~" H 5050 4050 50  0001 C CNN
+F 3 "http://www.farnell.com/datasheets/2049325.pdf" H 5050 4050 50  0001 C CNN
 	1    5050 4050
 	1    0    0    -1
@@
 	1    0    0    -1
 $EndComp
-Connection ~ 5050 3400
 $Comp
 L Connector_Generic:Conn_01x02 J2
 U 1 1 5DC5E6D5
-P 6200 3400
-F 0 "J2" H 6280 3392 50  0000 L CNN
-F 1 "Conn_01x02" H 6280 3301 50  0000 L CNN
-F 2 "Connector_PinHeader_2.54mm:PinHeader_1x02_P2.54mm_Vertical" H 6200 3400 50  0001 C CNN
-F 3 "~" H 6200 3400 50  0001 C CNN
-	1    6200 3400
+P 5850 3350
+F 0 "J2" H 5930 3342 50  0000 L CNN
+F 1 "Conn_01x02" H 5930 3251 50  0000 L CNN
+F 2 "Connector_PinHeader_2.54mm:PinHeader_1x02_P2.54mm_Vertical" H 5850 3350 50  0001 C CNN
+F 3 "http://www.farnell.com/datasheets/27856.pdf" H 5850 3350 50  0001 C CNN
+	1    5850 3350
 	1    0    0    -1
 $EndComp
@@
 F 1 "1.8k" H 5100 3050 50  0000 L CNN
 F 2 "Resistor_THT:R_Axial_DIN0207_L6.3mm_D2.5mm_P5.08mm_Vertical" H 5050 3100 50  0001 C CNN
-F 3 "~" H 5050 3100 50  0001 C CNN
+F 3 "http://www.farnell.com/datasheets/2049325.pdf" H 5050 3100 50  0001 C CNN
 	1    5050 3100
 	1    0    0    -1
 $EndComp
-Wire Wire Line
-	6000 3400 5750 3400
 Wire Wire Line
 	5050 4150 5050 4200
@@
 P 5500 4500
 F 0 "C2" V 5729 4500 50  0000 C CNN
-F 1 "40uF" V 5638 4500 50  0000 C CNN
+F 1 "470uF" V 5638 4500 50  0000 C CNN
 F 2 "Capacitor_THT:CP_Radial_D6.3mm_P2.50mm" H 5500 4500 50  0001 C CNN
-F 3 "~" H 5500 4500 50  0001 C CNN
+F 3 "http://www.farnell.com/datasheets/2321305.pdf" H 5500 4500 50  0001 C CNN
 	1    5500 4500
 	1    0    0    -1
@@
 F 1 "Conn_01x03" H 3868 3366 50  0000 C CNN
 F 2 "Connector_PinSocket_2.54mm:PinSocket_1x03_P2.54mm_Vertical" H 3950 3600 50  0001 C CNN
-F 3 "~" H 3950 3600 50  0001 C CNN
+F 3 "http://www.farnell.com/datasheets/27856.pdf" H 3950 3600 50  0001 C CNN
 	1    3950 3600
 	-1   0    0    1
 $EndComp
 Wire Wire Line
-	5050 3400 5550 3400
-Wire Wire Line
 	4150 3500 4350 3500
 Connection ~ 4750 2900
@@
 	5050 2900 5050 3000
 Wire Wire Line
-	5050 3200 5050 3400
+	5050 3200 5050 3350
 $Comp
 L power:GND #PWR04
 U 1 1 5E744DC4
-P 5900 3600
-F 0 "#PWR04" H 5900 3350 50  0001 C CNN
-F 1 "GND" H 5905 3427 50  0000 C CNN
-F 2 "" H 5900 3600 50  0001 C CNN
-F 3 "" H 5900 3600 50  0001 C CNN
-	1    5900 3600
-	1    0    0    -1
-$EndComp
-Wire Wire Line
-	5900 3500 5900 3600
+P 5550 3550
+F 0 "#PWR04" H 5550 3300 50  0001 C CNN
+F 1 "GND" H 5555 3377 50  0000 C CNN
+F 2 "" H 5550 3550 50  0001 C CNN
+F 3 "" H 5550 3550 50  0001 C CNN
+	1    5550 3550
+	1    0    0    -1
+$EndComp
+Wire Wire Line
+	5550 3450 5550 3550
 $Comp
 L Device:R_POT RV1
@@
 F 1 "R_POT" H 5430 4245 50  0000 R CNN
 F 2 "Potentiometer_SMD:Potentiometer_ACP_CA6-VSMD_Vertical" H 5500 4200 50  0001 C CNN
-F 3 "~" H 5500 4200 50  0001 C CNN
+F 3 "https://www.acptechnologies.com/wp-content/uploads/2017/06/01-ACP-CA6.pdf" H 5500 4200 50  0001 C CNN
 	1    5500 4200
 	-1   0    0    1
@@
 	5500 4400 5500 4350
 Wire Wire Line
-	5500 4650 4750 4650
+	5500 4650 5200 4650
 Connection ~ 4750 4650
 Wire Wire Line
@@
 L power:PWR_FLAG #FLG0102
 U 1 1 5E75B4F2
-P 5500 4650
-F 0 "#FLG0102" H 5500 4725 50  0001 C CNN
-F 1 "PWR_FLAG" H 5500 4823 50  0000 C CNN
-F 2 "" H 5500 4650 50  0001 C CNN
-F 3 "~" H 5500 4650 50  0001 C CNN
-	1    5500 4650
+P 5200 4650
+F 0 "#FLG0102" H 5200 4725 50  0001 C CNN
+F 1 "PWR_FLAG" H 5200 4823 50  0000 C CNN
+F 2 "" H 5200 4650 50  0001 C CNN
+F 3 "~" H 5200 4650 50  0001 C CNN
+	1    5200 4650
 	-1   0    0    1
 $EndComp
+Wire Wire Line
+	5500 3350 5650 3350
+Connection ~ 5050 3350
+Wire Wire Line
+	5050 3350 5050 3400
+Wire Wire Line
+	5050 3350 5300 3350
+Connection ~ 5200 4650
+Wire Wire Line
+	5200 4650 4750 4650
 $EndSCHEMATC

Commit message: Made PCB for Single_Transistor_AMP
Parts:
- C1, C3: footprint Capacitor_THT:CP_Radial_D6.3mm_P2.50mm -> Capacitor_SMD:C_0603_1608Metric
- R1, R2, R3, R4: footprint Resistor_THT:R_Axial_DIN0207_L6.3mm_D2.5mm_P5.08mm_Vertical -> Resistor_SMD:R_0603_1608Metric
Changed lines of the file:
@@
 F 0 "C1" V 4779 3600 50  0000 C CNN
 F 1 "10uF" V 4688 3600 50  0000 C CNN
-F 2 "Capacitor_THT:CP_Radial_D6.3mm_P2.50mm" H 4550 3600 50  0001 C CNN
+F 2 "Capacitor_SMD:C_0603_1608Metric" H 4550 3600 50  0001 C CNN
 F 3 "http://www.farnell.com/datasheets/1700589.pdf" H 4550 3600 50  0001 C CNN
 	1    4550 3600
@@
 F 0 "C3" V 5629 3350 50  0000 C CNN
 F 1 "10uF" V 5538 3350 50  0000 C CNN
-F 2 "Capacitor_THT:CP_Radial_D6.3mm_P2.50mm" H 5400 3350 50  0001 C CNN
+F 2 "Capacitor_SMD:C_0603_1608Metric" H 5400 3350 50  0001 C CNN
 F 3 "http://www.farnell.com/datasheets/1700589.pdf" H 5400 3350 50  0001 C CNN
 	1    5400 3350
@@
 F 0 "R1" H 4809 3396 50  0000 L CNN
 F 1 "39k" H 4809 3305 50  0000 L CNN
-F 2 "Resistor_THT:R_Axial_DIN0207_L6.3mm_D2.5mm_P5.08mm_Vertical" H 4750 3350 50  0001 C CNN
+F 2 "Resistor_SMD:R_0603_1608Metric" H 4750 3350 50  0001 C CNN
 F 3 "http://www.farnell.com/datasheets/2049325.pdf" H 4750 3350 50  0001 C CNN
 	1    4750 3350
@@
 F 0 "R2" H 4809 3896 50  0000 L CNN
 F 1 "10k" H 4809 3805 50  0000 L CNN
-F 2 "Resistor_THT:R_Axial_DIN0207_L6.3mm_D2.5mm_P5.08mm_Vertical" H 4750 3850 50  0001 C CNN
+F 2 "Resistor_SMD:R_0603_1608Metric" H 4750 3850 50  0001 C CNN
 F 3 "http://www.farnell.com/datasheets/2049325.pdf" H 4750 3850 50  0001 C CNN
 	1    4750 3850
@@
 F 0 "R4" H 5150 4000 50  0000 L CNN
 F 1 "560" H 5150 4100 50  0000 L CNN
-F 2 "Resistor_THT:R_Axial_DIN0207_L6.3mm_D2.5mm_P5.08mm_Vertical" H 5050 4050 50  0001 C CNN
+F 2 "Resistor_SMD:R_0603_1608Metric" H 5050 4050 50  0001 C CNN
 F 3 "http://www.farnell.com/datasheets/2049325.pdf" H 5050 4050 50  0001 C CNN
 	1    5050 4050
@@
 F 0 "R3" H 5100 3150 50  0000 L CNN
 F 1 "1.8k" H 5100 3050 50  0000 L CNN
-F 2 "Resistor_THT:R_Axial_DIN0207_L6.3mm_D2.5mm_P5.08mm_Vertical" H 5050 3100 50  0001 C CNN
+F 2 "Resistor_SMD:R_0603_1608Metric" H 5050 3100 50  0001 C CNN
 F 3 "http://www.farnell.com/datasheets/2049325.pdf" H 5050 3100 50  0001 C CNN
 	1    5050 3100
