File: Singe_transistor_AMP/Singe_transistor_AMP.kicad_pcb (KiCad board)
At the start: 2 copper layers, 0 parts

Commit message: Made PCB for Single_Transistor_AMP
Parts:
- added C1: 10uF, Capacitor_SMD:C_0603_1608Metric, F.Cu at (103.4, 97.9)
- added C2: 470uF, Capacitor_THT:CP_Radial_D6.3mm_P2.50mm, F.Cu at (116.9, 95.2)
- added C3: 10uF, Capacitor_SMD:C_0603_1608Metric, F.Cu at (111.5, 91.7)
- added J1: Conn_01x03, Connector_PinSocket_2.54mm:PinSocket_1x03_P2.54mm_Vertical, F.Cu at (99.6, 100.4)
- added J2: Conn_01x02, Connector_PinHeader_2.54mm:PinHeader_1x02_P2.54mm_Vertical, F.Cu at (122.5, 92.6)
- added Q1: NPN, Package_TO_SOT_THT:TO-92, F.Cu at (107.3, 95.2)
- added R1: 39k, Resistor_SMD:R_0603_1608Metric, F.Cu at (103.3, 94.6)
- added R2: 10k, Resistor_SMD:R_0603_1608Metric, F.Cu at (104.2, 100.4)
- added R3: 1.8k, Resistor_SMD:R_0603_1608Metric, F.Cu at (103.3, 91.6)
- added R4: 560, Resistor_SMD:R_0603_1608Metric, F.Cu at (107.7, 100.9)
- added RV1: R_POT, Potentiometer_SMD:Potentiometer_ACP_CA6-VSMD_Vertical, F.Cu at (116.2, 101.0)
Routing:
- net Net-(C3-Pad2): track 0.00 -> 11.0 mm
- net Net-(C1-Pad2): track 0.00 -> 10.7 mm
- net Net-(C3-Pad1): track 0.00 -> 10.3 mm
- net VDD: track 0.00 -> 8.45 mm
- net Net-(Q1-Pad3): track 0.00 -> 7.08 mm
- net Net-(C2-Pad1): track 0.00 -> 6.03 mm
- net Net-(C1-Pad1): track 0.00 -> 3.03 mm
- added copper zone on B.Cu, net GND
- added copper zone on F.Cu, net GND
Other:
- board outline added: 28 x 15 mm
- net class Default: via_dia 0.8 -> 0.6; via_drill 0.4 -> 0.3
- net class Power added: clearance 0.2, trace_width 0.4, via_dia 0.8, via_drill 0.4

Commit message: updated Single_transistor_AMP
Parts:
- moved R3 2.15 mm to (103.4, 93.8)
- moved C2 1.56 mm to (117.9, 94.0), turned to 180 degrees
- moved C3 0.91 mm to (111.6, 92.6)
- moved R2 0.87 mm to (103.4, 100.8), turned to 180 degrees
- moved R1 0.71 mm to (103.4, 95.3)
- moved R4 0.40 mm to (107.3, 100.9)
Routing:
- net VDD: track 8.45 -> 4.64 mm
- net Net-(C2-Pad1): track 6.03 -> 9.54 mm
- net Net-(C1-Pad2): track 10.7 -> 12.7 mm
- net Net-(C3-Pad2): track 11.0 -> 12.1 mm
- net Net-(C3-Pad1): track 10.3 -> 11.2 mm
