File: PWR_supply/ACtoDC.sch (KiCad schematic (older format))
At the start: 4 parts, among them J2 Conn_01x02, T1 Transformer_1P_1S

Commit message: updated Single_transistor_AMP
Other:
- note added: "10:1"
- note added: "Max 40 V\n"
Changed lines of the file:
@@
 	-1   0    0    1
 $EndComp
+Text Notes 4650 2500 0    50   ~ 0
+Max 40 V\n
+Text Notes 4050 3150 0    50   ~ 0
+10:1
 $EndSCHEMATC
